Commit message: more worlds and change in the tf for the camera (was wrong I think

File: acl_sim/urdf/asus_camera.urdf.xacro (robot description, xacro)
@@ -77,9 +77,11 @@
           <update_rate>60</update_rate>
           <camera>
-            <horizontal_fov>${62.8 * M_PI/180.0}</horizontal_fov>
+            <horizontal_fov>${90 * M_PI/180.0}</horizontal_fov>
             <image>
               <format>R8G8B8</format>
-              <width>120</width>
-              <height>90</height>
+<!--               <width>120</width>
+              <height>90</height> -->
+              <width>320</width>
+              <height>240</height>
             </image>
             <clip>

File: acl_sim/urdf/quadrotor_with_asus.urdf.xacro (robot description, xacro)
@@ -9,5 +9,6 @@
     <xacro:include filename="$(find acl_sim)/urdf/asus_camera.urdf.xacro" />
     <xacro:asus_camera name="camera" parent="base_link">
-      <origin xyz="0.1 0.0 -0.03" rpy="0 0 0"/>
+     <!-- <origin xyz="0.1 0.0 -0.03" rpy="0 0 0"/>-->
+         <origin xyz="0.1 0.0 0" rpy="0 0 0"/>
     </xacro:asus_camera>
        <!-- Sonar height sensor -->

Commit message: working with ns

File: acl_sim/urdf/asus_camera.urdf.xacro (robot description, xacro)
@@ -2,4 +2,6 @@
 <robot xmlns:xacro="http://www.ros.org/wiki/xacro">
     <xacro:property name="M_PI" value="3.1415926535897931" />
+    <xacro:property name="ns" value="$(arg ns)" />
+    <xacro:property name="tf_prefix" value="$(arg tf_prefix)" />
     <!--
      The asus_camera_model macro only adds the model, it does not also add

Commit message: done static exp comparison F U vs only F

File: acl_sim/urdf/asus_camera.urdf.xacro (robot description, xacro)
@@ -84,6 +84,6 @@
 <!--               <width>120</width>  320, 240
               <height>90</height> -->
-              <width>120</width>
-              <height>90</height>
+              <width>320</width>
+              <height>240</height>
             </image>
             <clip>

File: acl_sim/urdf/quadrotor_base.urdf.xacro (robot description, xacro)
@@ -14,5 +14,5 @@
         <origin xyz="0 0 0" rpy="0 0 0" />
         <geometry>
-          <mesh filename="package://acl_sim/meshes/quadrotor/quadrotor_base_2.dae"/>
+          <mesh filename="package://acl_sim/meshes/quadrotor/quadrotor_base_2.dae" scale="0.76 0.76 1"/>
         </geometry>
       </visual>
