Commit message: changed scale drone

File: acl_sim/urdf/quadrotor_base.urdf.xacro (robot description, xacro)
@@ -14,5 +14,5 @@
         <origin xyz="0 0 0" rpy="0 0 0" />
         <geometry>
-          <mesh filename="package://acl_sim/meshes/quadrotor/quadrotor_base_2.dae" scale="0.76 0.76 1"/>
+          <mesh filename="package://acl_sim/meshes/quadrotor/quadrotor_base_2.dae" scale="1.2 1.2 1"/>
         </geometry>
       </visual>
